Commit message: done

File: envs/robots/panda.urdf (robot description, URDF)
Before this commit: robot panda, 13 links, 12 joints
Joints:
- joint panda_joint1: origin xyz=-0.6 0 0.333 rpy=0 0 0 -> xyz=0.0 0 0.333 rpy=0 0 0

Commit message: local

File: envs/robots/panda.urdf (robot description, URDF)
Before this commit: robot panda, 13 links, 12 joints
Joints:
- joint panda_joint1: origin xyz=0.0 0 0.333 rpy=0 0 0 -> xyz=-0.6 0 0.333 rpy=0 0 0
