Commit message: done

File: envs/robots/jaco_robotiq.urdf (robot description, URDF)
Before this commit: robot j2s7s300, 19 links, 18 joints
Joints:
- joint robotiq_85_left_finger_joint: limit lower=-3.14 upper=3.14 velocity=100.0 -> lower=-3.14 upper=3.14 effort=50 velocity=100.0
- joint robotiq_85_left_finger_tip_joint: limit lower=-0.8 upper=0.1 velocity=100.0 -> lower=-0.8 upper=0.1 effort=50 velocity=100.0
- joint robotiq_85_left_inner_knuckle_joint: limit lower=-3.14 upper=3.14 velocity=100.0 -> lower=-3.14 upper=3.14 effort=50 velocity=100.0
- joint robotiq_85_left_knuckle_joint: limit lower=-0.7 upper=0.9 velocity=100.0 -> lower=-0.7 upper=0.9 effort=50 velocity=100.0
- joint robotiq_85_right_finger_joint: limit lower=-3.14 upper=3.14 velocity=100.0 -> lower=-3.14 upper=3.14 effort=50 velocity=100.0
- joint robotiq_85_right_finger_tip_joint: limit lower=-0.8 upper=0.1 velocity=100.0 -> lower=-0.8 upper=0.1 effort=50 velocity=100.0
- joint robotiq_85_right_inner_knuckle_joint: limit lower=-3.14 upper=3.14 velocity=100.0 -> lower=-3.14 upper=3.14 effort=50 velocity=100.0
- joint robotiq_85_right_knuckle_joint: limit lower=-0.7 upper=0.9 velocity=100.0 -> lower=-0.7 upper=0.9 effort=50 velocity=100.0
